File: pcb/mcu.kicad_sch (KiCad schematic)
At the start: 18 parts, among them J9 DNP, SW1 SKRKAEE020, SW2 SKRKAEE020, U7 ESP32-S3-WROOM-1

Commit message: Fixed ESP32-S3 footprint and symbol issues
Parts:
- U7: footprint RF_Module:ESP32-S3-WROOM-1 -> ESP32-S3:ESP32-S3-WROOM-1
Changed lines of the file:
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@@
+    (stroke (width 0) (type default))
+  )
+  (wire (pts (xy 77.47 143.51) (xy 91.44 143.51))
+    (stroke (width 0) (type default))
+  )
+  (wire (pts (xy 45.72 104.14) (xy 43.18 104.14))
+    (stroke (width 0) (type default))
+  )
+  (wire (pts (xy 49.53 143.51) (xy 48.26 143.51))
+    (stroke (width 0) (type default))
+  )
+  (wire (pts (xy 257.81 127) (xy 264.16 127))
+    (stroke (width 0) (type default))
+  )
+  (wire (pts (xy 205.74 62.23) (xy 224.79 62.23))
+    (stroke (width 0) (type default))
+  )
+  (wire (pts (xy 124.46 172.72) (xy 134.62 172.72))
+    (stroke (width 0) (type default))
+  )
+  (wire (pts (xy 29.21 16.51) (xy 48.26 16.51))
+    (stroke (width 0) (type default))
+  )
+  (wire (pts (xy 205.74 105.41) (xy 224.79 105.41))
+    (stroke (width 0) (type default))
+  )
+  (wire (pts (xy 57.15 104.14) (xy 64.77 104.14))
+    (stroke (width 0) (type default))
+  )
+  (wire (pts (xy 29.21 45.72) (xy 48.26 45.72))
+    (stroke (width 0) (type default))
+  )
+  (wire (pts (xy 205.74 87.63) (xy 224.79 87.63))
     (stroke (width 0) (type default))
   )
   (wire (pts (xy 160.02 135.89) (xy 160.02 138.43))
-    (stroke (width 0) (type default))
-  )
-  (wire (pts (xy 77.47 143.51) (xy 91.44 143.51))
-    (stroke (width 0) (type default))
-  )
-  (wire (pts (xy 45.72 104.14) (xy 43.18 104.14))
-    (stroke (width 0) (type default))
-  )
-  (wire (pts (xy 49.53 143.51) (xy 48.26 143.51))
-    (stroke (width 0) (type default))
-  )
-  (wire (pts (xy 257.81 127) (xy 264.16 127))
-    (stroke (width 0) (type default))
-  )
-  (wire (pts (xy 205.74 62.23) (xy 224.79 62.23))
-    (stroke (width 0) (type default))
-  )
-  (wire (pts (xy 124.46 172.72) (xy 134.62 172.72))
-    (stroke (width 0) (type default))
-  )
-  (wire (pts (xy 29.21 16.51) (xy 48.26 16.51))
-    (stroke (width 0) (type default))
-  )
-  (wire (pts (xy 205.74 105.41) (xy 224.79 105.41))
-    (stroke (width 0) (type default))
-  )
-  (wire (pts (xy 57.15 104.14) (xy 64.77 104.14))
-    (stroke (width 0) (type default))
-  )
-  (wire (pts (xy 29.21 45.72) (xy 48.26 45.72))
-    (stroke (width 0) (type default))
-  )
-  (wire (pts (xy 205.74 87.63) (xy 224.79 87.63))
     (stroke (width 0) (type default))
   )
@@
       (effects (font (size 1.27 1.27)) (justify left))
     )
-    (property "Footprint" "RF_Module:ESP32-S3-WROOM-1" (at 162.56 143.51 0)
-      (effects (font (size 1.27 1.27)) hide)
-    )
+    (property "Footprint" "ESP32-S3:ESP32-S3-WROOM-1" (at 162.56 143.51 0)
+      (effects (font (size 1.27 1.27)) hide)
+    )
