File: pcb/mcu.kicad_sch (KiCad schematic)
At the start: 18 parts, among them J9 DNP, SW1 SKRKAEE020, SW2 SKRKAEE020, U7 ESP32-S3-WROOM-1

Commit message: Added Testpoints on bottom side
Parts:
- added TP1: TB_SDA, TestPoint:TestPoint_Pad_D1.0mm, symbol Connector:TestPoint
- added TP2: TP_SCL, TestPoint:TestPoint_Pad_D1.0mm, symbol Connector:TestPoint
- added TP4: TP_EN_ESP, TestPoint:TestPoint_Pad_D1.0mm, symbol Connector:TestPoint
- added TP4: TP_GPIO0, TestPoint:TestPoint_Pad_D1.0mm, symbol Connector:TestPoint
Connections:
- net EN: now also TP4.1
- net GPIO_0: now also TP4.1
- net SCL: now also TP2.1
- net SDA: now also TP1.1
Changed lines of the file:
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@@
 (kicad_sch (version 20230121) (generator eeschema)
   (paper "A4")
+  (junction (at 248.92 127) (diameter 0) (color 0 0 0 0)
+  )
   (junction (at 160.02 38.1) (diameter 0) (color 0 0 0 0)
   )
@@
   )
   (junction (at 58.42 77.47) (diameter 0) (color 0 0 0 0)
+  )
+  (junction (at 250.19 120.65) (diameter 0) (color 0 0 0 0)
   )
   (no_connect (at 114.3 130.81))
@@
     (stroke (width 0) (type default))
   )
+  (wire (pts (xy 248.92 127) (xy 243.84 127))
+    (stroke (width 0) (type default))
+  )
+  (wire (pts (xy 250.19 113.03) (xy 250.19 120.65))
+    (stroke (width 0) (type default))
+  )
   (wire (pts (xy 142.24 165.1) (xy 124.46 165.1))
     (stroke (width 0) (type default))
@@
     (stroke (width 0) (type default))
   )
-  (wire (pts (xy 252.73 120.65) (xy 243.84 120.65))
+  (wire (pts (xy 252.73 120.65) (xy 250.19 120.65))
     (stroke (width 0) (type default))
   )
@@
     (stroke (width 0) (type default))
   )
+  (wire (pts (xy 250.19 120.65) (xy 243.84 120.65))
+    (stroke (width 0) (type default))
+  )
   (wire (pts (xy 90.17 48.26) (xy 90.17 50.8))
     (stroke (width 0) (type default))
@@
     (stroke (width 0) (type default))
   )
+  (wire (pts (xy 68.58 100.33) (xy 68.58 104.14))
+    (stroke (width 0) (type default))
+  )
   (wire (pts (xy 182.88 39.37) (xy 182.88 38.1))
     (stroke (width 0) (type default))
@@
     (stroke (width 0) (type default))
   )
-  (wire (pts (xy 57.15 104.14) (xy 64.77 104.14))
+  (wire (pts (xy 57.15 104.14) (xy 68.58 104.14))
     (stroke (width 0) (type default))
   )
@@
     (stroke (width 0) (type default))
   )
+  (wire (pts (xy 58.42 77.47) (xy 68.58 77.47))
+    (stroke (width 0) (type default))
+  )
+  (wire (pts (xy 248.92 127) (xy 248.92 138.43))
+    (stroke (width 0) (type default))
+  )
   (wire (pts (xy 160.02 38.1) (xy 160.02 54.61))
     (stroke (width 0) (type default))
@@
     (stroke (width 0) (type default))
   )
-  (wire (pts (xy 58.42 77.47) (xy 64.77 77.47))
-    (stroke (width 0) (type default))
-  )
   (wire (pts (xy 205.74 107.95) (xy 224.79 107.95))
     (stroke (width 0) (type default))
@@
     (stroke (width 0) (type default))
   )
+  (wire (pts (xy 255.27 137.16) (xy 255.27 138.43))
+    (stroke (width 0) (type default))
+  )
   (wire (pts (xy 29.21 29.21) (xy 48.26 29.21))
     (stroke (width 0) (type default))
   )
-  (wire (pts (xy 252.73 127) (xy 243.84 127))
+  (wire (pts (xy 252.73 127) (xy 248.92 127))
     (stroke (width 0) (type default))
   )
@@
     (stroke (width 0) (type default))
   )
+  (wire (pts (xy 68.58 74.93) (xy 68.58 77.47))
+    (stroke (width 0) (type default))
+  )
   (wire (pts (xy 205.74 67.31) (xy 233.68 67.31))
     (stroke (width 0) (type default))
@@
   )
   (wire (pts (xy 57.15 104.14) (xy 57.15 107.95))
+    (stroke (width 0) (type default))
+  )
+  (wire (pts (xy 255.27 138.43) (xy 248.92 138.43))
     (stroke (width 0) (type default))
   )
@@
     )
   )
+  (symbol (lib_id "Connector:TestPoint") (at 255.27 137.16 0) (unit 1)
+    (in_bom no) (on_board yes) (dnp no) (fields_autoplaced)
+    (property "Reference" "TP2" (at 257.81 132.588 0)
+      (effects (font (size 1.27 1.27)) (justify left))
+    )
+    (property "Value" "TP_SCL" (at 257.81 135.128 0)
+      (effects (font (size 1.27 1.27)) (justify left))
+    )
+    (property "Footprint" "TestPoint:TestPoint_Pad_D1.0mm" (at 260.35 137.16 0)
+      (effects (font (size 1.27 1.27)) hide)
+    )
+    (property "Datasheet" "~" (at 260.35 137.16 0)
+      (effects (font (size 1.27 1.27)) hide)
+    )
+    (pin "1")
+    (instances
+      (project "rep-trap-pcb"
+        (path "/b363dc8f-4a45-4779-a397-ccb82393dab8/eebb1d37-a01d-4adf-be70-a8e8f9293475/e7ccec12-46ad-495a-887c-7169982423a2"
+          (reference "TP2") (unit 1)
+        )
+      )
+    )
+  )
+  (symbol (lib_id "Connector:TestPoint") (at 68.58 74.93 0) (unit 1)
+    (in_bom no) (on_board yes) (dnp no) (fields_autoplaced)
+    (property "Reference" "TP4" (at 71.12 70.358 0)
+      (effects (font (size 1.27 1.27)) (justify left))
+    )
+    (property "Value" "TP_EN_ESP" (at 71.12 72.898 0)
+      (effects (font (size 1.27 1.27)) (justify left))
+    )
+    (property "Footprint" "TestPoint:TestPoint_Pad_D1.0mm" (at 73.66 74.93 0)
+      (effects (font (size 1.27 1.27)) hide)
+    )
+    (property "Datasheet" "~" (at 73.66 74.93 0)
+      (effects (font (size 1.27 1.27)) hide)
+    )
+    (pin "1")
+    (instances
+      (project "rep-trap-pcb"
+        (path "/b363dc8f-4a45-4779-a397-ccb82393dab8/eebb1d37-a01d-4adf-be70-a8e8f9293475/571cfc2c-17d3-4043-8736-10f73b37aef8"
+          (reference "TP4") (unit 1)
+        )
+        (path "/b363dc8f-4a45-4779-a397-ccb82393dab8/eebb1d37-a01d-4adf-be70-a8e8f9293475/e7ccec12-46ad-495a-887c-7169982423a2"
+          (reference "TP12") (unit 1)
+        )
+      )
+    )
+  )
   (symbol (lib_id "Device:C_Small") (at 168.91 41.91 0) (unit 1)
     (in_bom yes) (on_board yes) (dnp no) (fields_autoplaced)
@@
         (path "/c97100ff-06d7-45f1-a18e-c0adb622620f"
           (reference "R12") (unit 1)
+        )
+      )
+    )
+  )
+  (symbol (lib_id "Connector:TestPoint") (at 250.19 113.03 0) (unit 1)
+    (in_bom no) (on_board yes) (dnp no) (fields_autoplaced)
+    (property "Reference" "TP1" (at 252.73 108.458 0)
+      (effects (font (size 1.27 1.27)) (justify left))
+    )
+    (property "Value" "TB_SDA" (at 252.73 110.998 0)
+      (effects (font (size 1.27 1.27)) (justify left))
+    )
+    (property "Footprint" "TestPoint:TestPoint_Pad_D1.0mm" (at 255.27 113.03 0)
+      (effects (font (size 1.27 1.27)) hide)
+    )
+    (property "Datasheet" "~" (at 255.27 113.03 0)
+      (effects (font (size 1.27 1.27)) hide)
+    )
+    (pin "1")
+    (instances
+      (project "rep-trap-pcb"
+        (path "/b363dc8f-4a45-4779-a397-ccb82393dab8/eebb1d37-a01d-4adf-be70-a8e8f9293475/e7ccec12-46ad-495a-887c-7169982423a2"
+          (reference "TP1") (unit 1)
         )
       )
@@
         )
       )
+    )
+  )
+  (symbol (lib_id "Connector:TestPoint") (at 68.58 100.33 0) (unit 1)
+    (in_bom no) (on_board yes) (dnp no) (fields_autoplaced)
+    (property "Reference" "TP4" (at 71.12 95.758 0)
+      (effects (font (size 1.27 1.27)) (justify left))
+    )
+    (property "Value" "TP_GPIO0" (at 71.12 98.298 0)
+      (effects (font (size 1.27 1.27)) (justify left))
+    )
+    (property "Footprint" "TestPoint:TestPoint_Pad_D1.0mm" (at 73.66 100.33 0)
+      (effects (font (size 1.27 1.27)) hide)
+    )
+    (property "Datasheet" "~" (at 73.66 100.33 0)
+      (effects (font (size 1.27 1.27)) hide)
+    )
+    (pin "1")
+    (instances
+      (project "rep-trap-pcb"
+        (path "/b363dc8f-4a45-4779-a397-ccb82393dab8/eebb1d37-a01d-4adf-be70-a8e8f9293475/571cfc2c-17d3-4043-8736-10f73b37aef8"
+          (reference "TP4") (unit 1)
+        )
+        (path "/b363dc8f-4a45-4779-a397-ccb82393dab8/eebb1d37-a01d-4adf-be70-a8e8f9293475/e7ccec12-46ad-495a-887c-7169982423a2"
+          (reference "TP13") (unit 1)
+        )
+      )

Commit message: Update to use KiCad8
Parts:
- renumbered TP4 to TP12, TP4 to TP13
