File: pcb/tof-array.kicad_sch (KiCad schematic)
At the start: 20 parts, among them U1 VL53L4CDV0DH/1, U2 VL53L4CDV0DH/1, U3 VL53L4CDV0DH/1

Commit message: Refactored details component namings + bom excludings
Parts:
- C1, C4, C6: value 0.1uF -> 0.1µF
- C2, C3, C5: value 4.7uF -> 4.7µF
Changed lines of the file:
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@@
       (effects (font (size 1.27 1.27)) (justify left))
     )
-    (property "Value" "0.1uF" (at 267.7541 62.2436 0)
+    (property "Value" "0.1µF" (at 267.7541 62.2436 0)
       (effects (font (size 1.27 1.27)) (justify left))
     )
@@
       (effects (font (size 1.27 1.27)) (justify left))
     )
-    (property "Value" "0.1uF" (at 140.7541 92.7236 0)
+    (property "Value" "0.1µF" (at 140.7541 92.7236 0)
       (effects (font (size 1.27 1.27)) (justify left))
     )
@@
       (effects (font (size 1.27 1.27)) (justify left))
     )
-    (property "Value" "0.1uF" (at 139.4841 161.3036 0)
+    (property "Value" "0.1µF" (at 139.4841 161.3036 0)
       (effects (font (size 1.27 1.27)) (justify left))
     )
@@
       (effects (font (size 1.27 1.27)) (justify left))
     )
-    (property "Value" "4.7uF" (at 130.5941 92.7236 0)
+    (property "Value" "4.7µF" (at 130.5941 92.7236 0)
       (effects (font (size 1.27 1.27)) (justify left))
     )
@@
       (effects (font (size 1.27 1.27)) (justify left))
     )
-    (property "Value" "4.7uF" (at 257.5941 62.2436 0)
+    (property "Value" "4.7µF" (at 257.5941 62.2436 0)
       (effects (font (size 1.27 1.27)) (justify left))
     )
@@
       (effects (font (size 1.27 1.27)) (justify left))
     )
-    (property "Value" "4.7uF" (at 256.3241 130.8236 0)
+    (property "Value" "4.7µF" (at 256.3241 130.8236 0)
       (effects (font (size 1.27 1.27)) (justify left))
     )
@@
       (effects (font (size 1.27 1.27)) (justify left))
     )
-    (property "Value" "4.7uF" (at 129.3241 161.3036 0)
+    (property "Value" "4.7µF" (at 129.3241 161.3036 0)
       (effects (font (size 1.27 1.27)) (justify left))
     )
@@
       (effects (font (size 1.27 1.27)) (justify left))
     )
-    (property "Value" "0.1uF" (at 266.4841 130.8236 0)
-      (effects (font (size 1.27 1.27)) (justify left))
-    )
+    (property "Value" "0.1µF" (at 266.4841 130.8236 0)
+      (effects (font (size 1.27 1.27)) (justify left))
+    )

Commit message: refactored components and layout
Other:
- moved on the sheet: C1, C2, R1, R2, U1

Commit message: Replaced RP2040 with ESP32 + Schematics + Layouting
Other:
- moved on the sheet: C1, C2, R1, R2, U1

Commit message: Renamed tracks to fix ERC warnings
Changed lines of the file:
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@@
     (stroke (width 0) (type default))
   )
-  (label "~{INT_VL53_2}" (at 52.07 25.4 180) (fields_autoplaced)
+  (label "INT_VL53_2" (at 52.07 25.4 180) (fields_autoplaced)
     (effects (font (size 1.27 1.27)) (justify right bottom))
   )
-  (label "~{INT_VL53_4}" (at 52.07 30.48 180) (fields_autoplaced)
+  (label "INT_VL53_4" (at 52.07 30.48 180) (fields_autoplaced)
     (effects (font (size 1.27 1.27)) (justify right bottom))
   )
@@
     (effects (font (size 1.27 1.27)) (justify right bottom))
   )
-  (label "~{INT_VL53_3}" (at 242.57 68.58 180) (fields_autoplaced)
+  (label "INT_VL53_3" (at 242.57 68.58 180) (fields_autoplaced)
     (effects (font (size 1.27 1.27)) (justify right bottom))
   )
-  (label "~{INT_VL53_1}" (at 113.03 111.76 180) (fields_autoplaced)
+  (label "INT_VL53_1" (at 113.03 111.76 180) (fields_autoplaced)
     (effects (font (size 1.27 1.27)) (justify right bottom))
   )
@@
     (effects (font (size 1.27 1.27)) (justify left bottom))
   )
-  (label "~{INT_VL53_2}" (at 114.3 167.64 180) (fields_autoplaced)
+  (label "INT_VL53_2" (at 114.3 167.64 180) (fields_autoplaced)
     (effects (font (size 1.27 1.27)) (justify right bottom))
   )
-  (label "~{INT_VL53_1}" (at 52.07 22.86 180) (fields_autoplaced)
+  (label "INT_VL53_1" (at 52.07 22.86 180) (fields_autoplaced)
     (effects (font (size 1.27 1.27)) (justify right bottom))
   )
@@
     (effects (font (size 1.27 1.27)) (justify right bottom))
   )
-  (label "~{INT_VL53_3}" (at 187.96 90.17 0) (fields_autoplaced)
+  (label "INT_VL53_3" (at 187.96 90.17 0) (fields_autoplaced)
     (effects (font (size 1.27 1.27)) (justify left bottom))
   )
@@
     (effects (font (size 1.27 1.27)) (justify right bottom))
   )
-  (label "~{INT_VL53_1}" (at 58.42 133.35 0) (fields_autoplaced)
+  (label "INT_VL53_1" (at 58.42 133.35 0) (fields_autoplaced)
     (effects (font (size 1.27 1.27)) (justify left bottom))
   )
@@
     (effects (font (size 1.27 1.27)) (justify left bottom))
   )
-  (label "~{INT_VL53_2}" (at 59.69 189.23 0) (fields_autoplaced)
+  (label "INT_VL53_2" (at 59.69 189.23 0) (fields_autoplaced)
     (effects (font (size 1.27 1.27)) (justify left bottom))
   )
@@
     (effects (font (size 1.27 1.27)) (justify right bottom))
   )
-  (label "~{INT_VL53_3}" (at 52.07 27.94 180) (fields_autoplaced)
+  (label "INT_VL53_3" (at 52.07 27.94 180) (fields_autoplaced)
     (effects (font (size 1.27 1.27)) (justify right bottom))
   )
-  (label "~{INT_VL53_4}" (at 186.69 158.75 0) (fields_autoplaced)
+  (label "INT_VL53_4" (at 186.69 158.75 0) (fields_autoplaced)
     (effects (font (size 1.27 1.27)) (justify left bottom))
   )
@@
     (effects (font (size 1.27 1.27)) (justify left bottom))
   )
-  (label "~{INT_VL53_4}" (at 241.3 137.16 180) (fields_autoplaced)
+  (label "INT_VL53_4" (at 241.3 137.16 180) (fields_autoplaced)
     (effects (font (size 1.27 1.27)) (justify right bottom))
   )

Commit message: Changed net names to match functionallity of active low
Connections:
- net INT_VL53_1 renamed ~{INT_VL53_1}
- net INT_VL53_2 renamed ~{INT_VL53_2}
- net INT_VL53_3 renamed ~{INT_VL53_3}
- net INT_VL53_4 renamed ~{INT_VL53_4}
- net XSHUT_VL53_1 renamed ~{XSHUT_VL53_1}
- net XSHUT_VL53_2 renamed ~{XSHUT_VL53_2}
- net XSHUT_VL53_3 renamed ~{XSHUT_VL53_3}
- net XSHUT_VL53_4 renamed ~{XSHUT_VL53_4}
Changed lines of the file:
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@@
     (stroke (width 0) (type default))
   )
-  (label "INT_VL53_2" (at 52.07 25.4 180) (fields_autoplaced)
+  (label "~{INT_VL53_2}" (at 52.07 25.4 180) (fields_autoplaced)
     (effects (font (size 1.27 1.27)) (justify right bottom))
   )
-  (label "INT_VL53_4" (at 52.07 30.48 180) (fields_autoplaced)
+  (label "~{INT_VL53_4}" (at 52.07 30.48 180) (fields_autoplaced)
     (effects (font (size 1.27 1.27)) (justify right bottom))
   )
@@
     (effects (font (size 1.27 1.27)) (justify right bottom))
   )
-  (label "INT_VL53_3" (at 242.57 68.58 180) (fields_autoplaced)
+  (label "~{INT_VL53_3}" (at 242.57 68.58 180) (fields_autoplaced)
     (effects (font (size 1.27 1.27)) (justify right bottom))
   )
-  (label "INT_VL53_1" (at 113.03 111.76 180) (fields_autoplaced)
+  (label "~{INT_VL53_1}" (at 113.03 111.76 180) (fields_autoplaced)
     (effects (font (size 1.27 1.27)) (justify right bottom))
   )
-  (label "XSHUT_VL53_2" (at 34.29 165.1 0) (fields_autoplaced)
+  (label "~{XSHUT_VL53_2}" (at 34.29 165.1 0) (fields_autoplaced)
     (effects (font (size 1.27 1.27)) (justify left bottom))
   )
-  (label "XSHUT_VL53_2" (at 59.69 182.88 0) (fields_autoplaced)
+  (label "~{XSHUT_VL53_2}" (at 59.69 182.88 0) (fields_autoplaced)
     (effects (font (size 1.27 1.27)) (justify left bottom))
   )
-  (label "INT_VL53_2" (at 114.3 167.64 180) (fields_autoplaced)
+  (label "~{INT_VL53_2}" (at 114.3 167.64 180) (fields_autoplaced)
     (effects (font (size 1.27 1.27)) (justify right bottom))
   )
-  (label "INT_VL53_1" (at 52.07 22.86 180) (fields_autoplaced)
+  (label "~{INT_VL53_1}" (at 52.07 22.86 180) (fields_autoplaced)
     (effects (font (size 1.27 1.27)) (justify right bottom))
   )
-  (label "XSHUT_VL53_4" (at 161.29 134.62 0) (fields_autoplaced)
+  (label "~{XSHUT_VL53_4}" (at 161.29 134.62 0) (fields_autoplaced)
     (effects (font (size 1.27 1.27)) (justify left bottom))
   )
@@
     (effects (font (size 1.27 1.27)) (justify right bottom))
   )
-  (label "INT_VL53_3" (at 187.96 90.17 0) (fields_autoplaced)
+  (label "~{INT_VL53_3}" (at 187.96 90.17 0) (fields_autoplaced)
     (effects (font (size 1.27 1.27)) (justify left bottom))
   )
-  (label "XSHUT_VL53_4" (at 52.07 40.64 180) (fields_autoplaced)
+  (label "~{XSHUT_VL53_4}" (at 52.07 40.64 180) (fields_autoplaced)
     (effects (font (size 1.27 1.27)) (justify right bottom))
   )
@@
     (effects (font (size 1.27 1.27)) (justify right bottom))
   )
-  (label "INT_VL53_1" (at 58.42 133.35 0) (fields_autoplaced)
+  (label "~{INT_VL53_1}" (at 58.42 133.35 0) (fields_autoplaced)
     (effects (font (size 1.27 1.27)) (justify left bottom))
   )
-  (label "XSHUT_VL53_4" (at 186.69 152.4 0) (fields_autoplaced)
+  (label "~{XSHUT_VL53_4}" (at 186.69 152.4 0) (fields_autoplaced)
     (effects (font (size 1.27 1.27)) (justify left bottom))
   )
-  (label "XSHUT_VL53_1" (at 52.07 33.02 180) (fields_autoplaced)
+  (label "~{XSHUT_VL53_1}" (at 52.07 33.02 180) (fields_autoplaced)
     (effects (font (size 1.27 1.27)) (justify right bottom))
   )
@@
     (effects (font (size 1.27 1.27)) (justify right bottom))
   )
-  (label "XSHUT_VL53_3" (at 162.56 66.04 0) (fields_autoplaced)
+  (label "~{XSHUT_VL53_3}" (at 162.56 66.04 0) (fields_autoplaced)
     (effects (font (size 1.27 1.27)) (justify left bottom))
   )
@@
     (effects (font (size 1.27 1.27)) (justify right bottom))
   )
-  (label "XSHUT_VL53_3" (at 187.96 83.82 0) (fields_autoplaced)
+  (label "~{XSHUT_VL53_3}" (at 187.96 83.82 0) (fields_autoplaced)
     (effects (font (size 1.27 1.27)) (justify left bottom))
   )
-  (label "INT_VL53_2" (at 59.69 189.23 0) (fields_autoplaced)
+  (label "~{INT_VL53_2}" (at 59.69 189.23 0) (fields_autoplaced)
     (effects (font (size 1.27 1.27)) (justify left bottom))
   )
@@
     (effects (font (size 1.27 1.27)) (justify right bottom))
   )
-  (label "INT_VL53_3" (at 52.07 27.94 180) (fields_autoplaced)
+  (label "~{INT_VL53_3}" (at 52.07 27.94 180) (fields_autoplaced)
     (effects (font (size 1.27 1.27)) (justify right bottom))
   )
-  (label "INT_VL53_4" (at 186.69 158.75 0) (fields_autoplaced)
+  (label "~{INT_VL53_4}" (at 186.69 158.75 0) (fields_autoplaced)
     (effects (font (size 1.27 1.27)) (justify left bottom))
   )
-  (label "XSHUT_VL53_1" (at 58.42 127 0) (fields_autoplaced)
+  (label "~{XSHUT_VL53_1}" (at 58.42 127 0) (fields_autoplaced)
     (effects (font (size 1.27 1.27)) (justify left bottom))
   )
-  (label "INT_VL53_4" (at 241.3 137.16 180) (fields_autoplaced)
+  (label "~{INT_VL53_4}" (at 241.3 137.16 180) (fields_autoplaced)
     (effects (font (size 1.27 1.27)) (justify right bottom))
   )
-  (label "XSHUT_VL53_3" (at 52.07 38.1 180) (fields_autoplaced)
+  (label "~{XSHUT_VL53_3}" (at 52.07 38.1 180) (fields_autoplaced)
     (effects (font (size 1.27 1.27)) (justify right bottom))
   )
-  (label "XSHUT_VL53_2" (at 52.07 35.56 180) (fields_autoplaced)
+  (label "~{XSHUT_VL53_2}" (at 52.07 35.56 180) (fields_autoplaced)
     (effects (font (size 1.27 1.27)) (justify right bottom))
   )
-  (label "XSHUT_VL53_1" (at 33.02 109.22 0) (fields_autoplaced)
+  (label "~{XSHUT_VL53_1}" (at 33.02 109.22 0) (fields_autoplaced)
     (effects (font (size 1.27 1.27)) (justify left bottom))
   )
-  (hierarchical_label "XSHUT_VL53_4" (shape input) (at 33.02 40.64 180) (fields_autoplaced)
+  (hierarchical_label "~{XSHUT_VL53_4}" (shape input) (at 33.02 40.64 180) (fields_autoplaced)
     (effects (font (size 1.27 1.27)) (justify right))
   )
-  (hierarchical_label "INT_VL53_4" (shape input) (at 33.02 30.48 180) (fields_autoplaced)
+  (hierarchical_label "~{INT_VL53_4}" (shape input) (at 33.02 30.48 180) (fields_autoplaced)
     (effects (font (size 1.27 1.27)) (justify right))
   )
-  (hierarchical_label "INT_VL53_1" (shape input) (at 33.02 22.86 180) (fields_autoplaced)
+  (hierarchical_label "~{INT_VL53_1}" (shape input) (at 33.02 22.86 180) (fields_autoplaced)
     (effects (font (size 1.27 1.27)) (justify right))
   )
@@
     (effects (font (size 1.27 1.27)) (justify right))
   )
-  (hierarchical_label "INT_VL53_2" (shape input) (at 33.02 25.4 180) (fields_autoplaced)
+  (hierarchical_label "~{INT_VL53_2}" (shape input) (at 33.02 25.4 180) (fields_autoplaced)
     (effects (font (size 1.27 1.27)) (justify right))
   )
-  (hierarchical_label "XSHUT_VL53_1" (shape input) (at 33.02 33.02 180) (fields_autoplaced)
+  (hierarchical_label "~{XSHUT_VL53_1}" (shape input) (at 33.02 33.02 180) (fields_autoplaced)
     (effects (font (size 1.27 1.27)) (justify right))
   )
-  (hierarchical_label "INT_VL53_3" (shape input) (at 33.02 27.94 180) (fields_autoplaced)
+  (hierarchical_label "~{INT_VL53_3}" (shape input) (at 33.02 27.94 180) (fields_autoplaced)
     (effects (font (size 1.27 1.27)) (justify right))
   )
@@
     (effects (font (size 1.27 1.27)) (justify right))
   )
-  (hierarchical_label "XSHUT_VL53_3" (shape input) (at 33.02 38.1 180) (fields_autoplaced)
+  (hierarchical_label "~{XSHUT_VL53_3}" (shape input) (at 33.02 38.1 180) (fields_autoplaced)
     (effects (font (size 1.27 1.27)) (justify right))
   )
-  (hierarchical_label "XSHUT_VL53_2" (shape input) (at 33.02 35.56 180) (fields_autoplaced)
+  (hierarchical_label "~{XSHUT_VL53_2}" (shape input) (at 33.02 35.56 180) (fields_autoplaced)
     (effects (font (size 1.27 1.27)) (justify right))
   )

Commit message: Added Testpoints on bottom side
Parts:
- added TP10: TP_XSHUT_3, TestPoint:TestPoint_Pad_D1.0mm, symbol Connector:TestPoint
- added TP11: TP_INT_3, TestPoint:TestPoint_Pad_D1.0mm, symbol Connector:TestPoint
- added TP4: TP_XSHUT_1, TestPoint:TestPoint_Pad_D1.0mm, symbol Connector:TestPoint
- added TP5: TP_INT_1, TestPoint:TestPoint_Pad_D1.0mm, symbol Connector:TestPoint
- added TP6: TP_XSHUT_2, TestPoint:TestPoint_Pad_D1.0mm, symbol Connector:TestPoint
- added TP7: TP_INT_2, TestPoint:TestPoint_Pad_D1.0mm, symbol Connector:TestPoint
- added TP8: TP_XSHUT_4, TestPoint:TestPoint_Pad_D1.0mm, symbol Connector:TestPoint
- added TP9: TP_INT_4, TestPoint:TestPoint_Pad_D1.0mm, symbol Connector:TestPoint
Connections:
- net ~{INT_VL53_1}: now also TP5.1
- net ~{INT_VL53_2}: now also TP7.1
- net ~{INT_VL53_3}: now also TP11.1
- net ~{INT_VL53_4}: now also TP9.1
- net ~{XSHUT_VL53_1}: now also TP4.1
- net ~{XSHUT_VL53_2}: now also TP6.1
- net ~{XSHUT_VL53_3}: now also TP10.1
- net ~{XSHUT_VL53_4}: now also TP8.1

Commit message: Update to use KiCad8
Parts:
- renumbered C5 to C10, C6 to C11, C6 to C12, C3 to C5, C2 to C6, C4 to C7, C1 to C8, C5 to C9, R2 to R10, R5 to R11, R6 to R12, R5 to R13, R6 to R14, R3 to R7, R4 to R8, R1 to R9, U2 to U3, U1 to U4, U3 to U5, U3 to U6
