File: pcb/main.kicad_sch (KiCad schematic)
At the start: 14 parts, among them IC1 DRV5032FBLPG, J3 SJ-3541AS-SMT-TR-67

Commit message: PCB update
Parts:
- removed JP3: jumper, Jumper:SolderJumper-2_P1.3mm_Bridged_RoundedPad1.0x1.5mm, symbol Jumper:SolderJumper_2_Bridged
- J3: value SJ-3541AS-SMT-TR-67 -> PJ-3254A-SMT; Alternative: (none) -> SJ-3541AS-SMT-TR-67
Connections:
- no-connect marks 3 -> 4
Changed lines of the file:
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@@
+	)
+	(no_connect
+		(at 251.46 116.84)
 	)
 	(no_connect
@@
 	(wire
 		(pts
-			(xy 267.97 116.84) (xy 273.05 116.84)
-		)
-		(stroke
-			(width 0)
-			(type default)
-		)
-	)
-	(wire
-		(pts
 			(xy 69.85 74.93) (xy 87.63 74.93)
 		)
@@
 		(pts
 			(xy 125.73 44.45) (xy 143.51 44.45)
-		)
-		(stroke
-			(width 0)
-			(type default)
-		)
-	)
-	(wire
-		(pts
-			(xy 251.46 116.84) (xy 260.35 116.84)
 		)
 		(stroke
@@
 		)
 	)
-	(label "RING"
-		(at 273.05 116.84 180)
-		(fields_autoplaced yes)
-		(effects
-			(font
-				(size 1.27 1.27)
-			)
-			(justify right bottom)
-		)
-	)
 	(label "END"
 		(at 260.35 99.06 180)
@@
 	)
 	(symbol
-		(lib_id "Jumper:SolderJumper_2_Bridged")
-		(at 264.16 116.84 0)
-		(unit 1)
-		(exclude_from_sim no)
-		(in_bom no)
-		(on_board yes)
-		(dnp no)
-		(fields_autoplaced yes)
-		(property "Reference" "JP3"
-			(at 264.16 110.49 0)
-			(effects
-				(font
-					(size 1.27 1.27)
-				)
-			)
-		)
-		(property "Value" "jumper"
-			(at 264.16 113.03 0)
-			(effects
-				(font
-					(size 1.27 1.27)
-				)
-			)
-		)
-		(property "Footprint" "Jumper:SolderJumper-2_P1.3mm_Bridged_RoundedPad1.0x1.5mm"
-			(at 264.16 116.84 0)
-			(effects
-				(font
-					(size 1.27 1.27)
-				)
-				(hide yes)
-			)
-		)
-		(property "Datasheet" "~"
-			(at 264.16 116.84 0)
-			(effects
-				(font
-					(size 1.27 1.27)
-				)
-				(hide yes)
-			)
-		)
-		(property "Description" ""
-			(at 264.16 116.84 0)
-			(effects
-				(font
-					(size 1.27 1.27)
-				)
-				(hide yes)
-			)
-		)
-		(pin "1"
-		)
-		(pin "2"
-		)
-		(instances
-			(project "rep-trap-pcb"
-				(path "/b363dc8f-4a45-4779-a397-ccb82393dab8/eebb1d37-a01d-4adf-be70-a8e8f9293475"
-					(reference "JP3")
-					(unit 1)
-				)
-			)
-		)
-	)
-	(symbol
 		(lib_id "Device:R_Small")
 		(at 204.47 143.51 90)
@@
 			)
 		)
-		(property "Value" "SJ-3541AS-SMT-TR-67"
+		(property "Value" "PJ-3254A-SMT"
 			(at 233.7435 93.98 0)
 			(effects
@@
 				(hide yes)
 			)
+		)
+		(property "Alternative:" "SJ-3541AS-SMT-TR-67"
+			(at 233.68 109.22 0)
+			(effects
+				(font
+					(size 1.27 1.27)
+				)
+				(hide yes)
+			)
